Commit message: Added a motor controller interface for the smile mobile simulation to accept PWM inputs. Also colored the robot.

File: smile_mobile_sim_ws/src/smile_mobile_description/urdf/smile.urdf.xacro (robot description, xacro)
@@ -1,9 +1,9 @@
 <?xml version="1.0"?>
 <robot name="smile" xmlns:xacro="http//www.ros.org/wiki/xacro">
-  <!--Chasis Dimension [9" 10.5" 1.32"]-->
-  <xacro:property name="chasis_width" value="0.2286"/>
-  <xacro:property name="chasis_length" value="0.2667"/>
-  <xacro:property name="chasis_height" value="0.033528"/>
-  <xacro:property name="chasis_mass" value="0.33"/>
+  <!--chassis Dimension [9" 10.5" 1.32"]-->
+  <xacro:property name="chassis_width" value="0.2286"/>
+  <xacro:property name="chassis_length" value="0.2667"/>
+  <xacro:property name="chassis_height" value="0.033528"/>
+  <xacro:property name="chassis_mass" value="0.33"/>
   <xacro:property name="wheel_radius" value="0.06858"/>
   <xacro:property name="wheel_width" value="0.0254"/>
@@ -12,24 +12,24 @@
   <xacro:property name="pi_div_2" value="1.57075"/>
   <link name="base_link"/>
-  <!-- Chasis -->
-  <link name="chasis">
-    <visual>
-      <geometry>
-        <box size="${chasis_width} ${chasis_length} ${chasis_height}"/>
-      </geometry>
-    </visual>
-    <collision>
-      <geometry>
-        <box size="${chasis_width} ${chasis_length} ${chasis_height}"/>
-      </geometry>
-    </collision>
-    <inertial>
-      <mass value="${chasis_mass}"/>
-      <inertia ixx="0.01" ixy="0.0" ixz="0.0" iyy="0.01" iyz="0.0" izz="0.01"/>
-    </inertial>
-  </link>
-  <joint name="base_link_to_chasis" type="fixed">
+  <!-- chassis -->
+  <link name="chassis">
+    <visual>
+      <geometry>
+        <box size="${chassis_width} ${chassis_length} ${chassis_height}"/>
+      </geometry>
+    </visual>
+    <collision>
+      <geometry>
+        <box size="${chassis_width} ${chassis_length} ${chassis_height}"/>
+      </geometry>
+    </collision>
+    <inertial>
+      <mass value="${chassis_mass}"/>
+      <inertia ixx="0.001" ixy="0.0" ixz="0.0" iyy="0.001" iyz="0.0" izz="0.001"/>
+    </inertial>
+  </link>
+  <joint name="base_link_to_chassis" type="fixed">
     <parent link="base_link"/>
-    <child link="chasis"/>
+    <child link="chassis"/>
   </joint>
   <!-- Left Front Wheel-->
@@ -54,7 +54,7 @@
   </link>
   <joint name="base_to_left_front_wheel" type="continuous">
-    <parent link="chasis"/>
+    <parent link="chassis"/>
     <child link="left_front_wheel"/>
-    <origin xyz="${-1 * chasis_width / 2} ${(chasis_length / 2) - wheel_pos_offset} 0 "/>
+    <origin xyz="${-1 * chassis_width / 2} ${(chassis_length / 2) - wheel_pos_offset} 0 "/>
   </joint>
     <!-- Right Front Wheel-->
@@ -79,7 +79,7 @@
   </link>
   <joint name="base_to_right_front_wheel" type="continuous">
-    <parent link="chasis"/>
+    <parent link="chassis"/>
     <child link="right_front_wheel"/>
-    <origin xyz="${chasis_width / 2} ${(chasis_length / 2) - wheel_pos_offset} 0 "/>
+    <origin xyz="${chassis_width / 2} ${(chassis_length / 2) - wheel_pos_offset} 0 "/>
   </joint>
     <!-- Left Back Wheel-->
@@ -104,7 +104,7 @@
   </link>
   <joint name="base_to_left_back_wheel" type="continuous">
-    <parent link="chasis"/>
+    <parent link="chassis"/>
     <child link="left_back_wheel"/>
-    <origin xyz="${-1 * chasis_width / 2} ${-1 *(chasis_length / 2) + wheel_pos_offset} 0 "/>
+    <origin xyz="${-1 * chassis_width / 2} ${-1 *(chassis_length / 2) + wheel_pos_offset} 0 "/>
   </joint>
   <!-- Right Back Wheel -->
@@ -129,10 +129,10 @@
   </link>
   <joint name="base_to_right_back_wheel" type="continuous">
-    <parent link="chasis"/>
+    <parent link="chassis"/>
     <child link="right_back_wheel"/>
-    <origin xyz="${chasis_width / 2} ${-1*(chasis_length / 2) + wheel_pos_offset} 0 "/>
+    <origin xyz="${chassis_width / 2} ${-1*(chassis_length / 2) + wheel_pos_offset} 0 "/>
   </joint>
   <!-- Gazebo References for URDF model
-  <gazebo reference="chasis">
+  <gazebo reference="chassis">
     <material>Gazebo/FlatBlack</material>
   </gazebo>
@@ -183,3 +183,19 @@
   </plugin>
 </gazebo>
+<!--Add colors for gazebo to each part of the vehicle-->
+<gazebo reference="chassis">
+  <material>Gazebo/Red</material>
+</gazebo>
+<gazebo reference="left_front_wheel">
+  <material>Gazebo/Grey</material>
+</gazebo>
+<gazebo reference="left_back_wheel">
+  <material>Gazebo/Grey</material>
+</gazebo>
+<gazebo reference="right_front_wheel">
+  <material>Gazebo/Grey</material>
+</gazebo>
+<gazebo reference="right_back_wheel">
+  <material>Gazebo/Grey</material>
+</gazebo>
 </robot>

Commit message: Minimized the issue with the robot flipping when changing the velocity too fast. Simply made the robot weigh more and added more damping to the joints.

File: smile_mobile_sim_ws/src/smile_mobile_description/urdf/smile.urdf.xacro (robot description, xacro)
@@ -5,9 +5,9 @@
   <xacro:property name="chassis_length" value="0.2667"/>
   <xacro:property name="chassis_height" value="0.033528"/>
-  <xacro:property name="chassis_mass" value="0.33"/>
+  <xacro:property name="chassis_mass" value="1.0"/>
   <xacro:property name="wheel_radius" value="0.06858"/>
   <xacro:property name="wheel_width" value="0.0254"/>
   <xacro:property name="wheel_pos_offset" value=".0254"/>
-  <xacro:property name="wheel_mass" value="0.05"/>
+  <xacro:property name="wheel_mass" value="0.5"/>
   <xacro:property name="pi_div_2" value="1.57075"/>
   <link name="base_link"/>
@@ -26,5 +26,8 @@
     <inertial>
       <mass value="${chassis_mass}"/>
-      <inertia ixx="0.001" ixy="0.0" ixz="0.0" iyy="0.001" iyz="0.0" izz="0.001"/>
+      <inertia
+        ixx="${chassis_mass / 12.0 * (chassis_length*chassis_length + chassis_height*chassis_height)}" ixy="0.0" ixz="0.0"
+        iyy="${chassis_mass / 12.0 * (chassis_width*chassis_width + chassis_height*chassis_height)}" iyz="0.0"
+        izz="${chassis_mass / 12.0 * (chassis_width*chassis_width + chassis_length*chassis_length)}"/>
     </inertial>
   </link>
@@ -49,5 +52,8 @@
     <inertial>
       <mass value="${wheel_mass}"/>
-      <inertia ixx="0.01" ixy="0.0" ixz="0.0" iyy="0.01" iyz="0.0" izz="0.01"/>
+      <inertia
+        ixx="${wheel_mass / 2.0 * wheel_radius * wheel_radius}" ixy="0.0" ixz="0.0"
+        iyy="0.01" iyz="0.0"
+        izz="0.01"/>
       <origin rpy="0 ${pi_div_2} 0" xyz="${-1 * wheel_width / 2} 0 0"/>
     </inertial>
@@ -57,4 +63,5 @@
     <child link="left_front_wheel"/>
     <origin xyz="${-1 * chassis_width / 2} ${(chassis_length / 2) - wheel_pos_offset} 0 "/>
+    <dynamics damping="1.5"/>
   </joint>
     <!-- Right Front Wheel-->
@@ -74,5 +81,8 @@
     <inertial>
       <mass value="${wheel_mass}"/>
-      <inertia ixx="0.01" ixy="0.0" ixz="0.0" iyy="0.01" iyz="0.0" izz="0.01"/>
+      <inertia
+        ixx="${wheel_mass / 2.0 * wheel_radius * wheel_radius}" ixy="0.0" ixz="0.0"
+        iyy="0.01" iyz="0.0"
+        izz="0.01"/>
       <origin rpy="0 ${pi_div_2} 0" xyz="${wheel_width / 2} 0 0"/>
     </inertial>
@@ -82,4 +92,5 @@
     <child link="right_front_wheel"/>
     <origin xyz="${chassis_width / 2} ${(chassis_length / 2) - wheel_pos_offset} 0 "/>
+    <dynamics damping="1.5"/>
   </joint>
     <!-- Left Back Wheel-->
@@ -99,5 +110,8 @@
     <inertial>
       <mass value="${wheel_mass}"/>
-      <inertia ixx="0.01" ixy="0.0" ixz="0.0" iyy="0.01" iyz="0.0" izz="0.01"/>
+      <inertia
+        ixx="${wheel_mass / 2.0 * wheel_radius * wheel_radius}" ixy="0.0" ixz="0.0"
+        iyy="0.01" iyz="0.0"
+        izz="0.01"/>
       <origin rpy="0 ${pi_div_2} 0" xyz="${-1 * wheel_width / 2} 0 0"/>
     </inertial>
@@ -107,4 +121,5 @@
     <child link="left_back_wheel"/>
     <origin xyz="${-1 * chassis_width / 2} ${-1 *(chassis_length / 2) + wheel_pos_offset} 0 "/>
+    <dynamics damping="1.5"/>
   </joint>
   <!-- Right Back Wheel -->
@@ -124,5 +139,8 @@
     <inertial>
       <mass value="${wheel_mass}"/>
-      <inertia ixx="0.01" ixy="0.0" ixz="0.0" iyy="0.01" iyz="0.0" izz="0.01"/>
+      <inertia
+        ixx="${wheel_mass / 2.0 * wheel_radius * wheel_radius}" ixy="0.0" ixz="0.0"
+        iyy="0.01" iyz="0.0"
+        izz="0.01"/>
       <origin rpy="0 ${pi_div_2} 0" xyz="${wheel_width / 2} 0 0"/>
     </inertial>
@@ -132,4 +150,13 @@
     <child link="right_back_wheel"/>
     <origin xyz="${chassis_width / 2} ${-1*(chassis_length / 2) + wheel_pos_offset} 0 "/>
+    <dynamics damping="1.5"/>
+  </joint>
+  <!--A small link to connect the IMU to the chassis-->
+  <link name="imu_link">
+  </link>
+  <joint name="chassis_to_imu_link" type="fixed">
+    <parent link="chassis"/>
+    <child link="imu_link"/>
+    <origin xyz="0.0 0.0 0.0"/>
   </joint>
   <!-- Gazebo References for URDF model
@@ -189,13 +216,42 @@
 <gazebo reference="left_front_wheel">
   <material>Gazebo/Grey</material>
+  <mu1>0.5</mu1>
+  <mu2>0.5</mu2>
 </gazebo>
 <gazebo reference="left_back_wheel">
   <material>Gazebo/Grey</material>
+  <mu1>0.5</mu1>
+  <mu2>0.5</mu2>
 </gazebo>
 <gazebo reference="right_front_wheel">
   <material>Gazebo/Grey</material>
+  <mu1>0.5</mu1>
+  <mu2>0.5</mu2>
 </gazebo>
 <gazebo reference="right_back_wheel">
   <material>Gazebo/Grey</material>
+  <mu1>0.5</mu1>
+  <mu2>0.5</mu2>
+</gazebo>
+<!--IMU Sensor Plugin-->
+<gazebo reference="imu_link">
+  <gravity>true</gravity>
+  <sensor name="imu_sensor" type="imu">
+    <always_on>true</always_on>
+    <update_rate>100</update_rate>
+    <visualize>true</visualize>
+    <topic>__default_topic__</topic>
+    <plugin filename="libgazebo_ros_imu_sensor.so" name="imu_plugin">
+      <topicName>imu</topicName>
+      <bodyName>imu_link</bodyName>
+      <updateRateHZ>10.0</updateRateHZ>
+      <gaussianNoise>0.0</gaussianNoise>
+      <xyzOffset>0 0 0</xyzOffset>
+      <rpyOffset>0 0 0</rpyOffset>
+      <frameName>imu_link</frameName>
+      <initialOrientationAsReference>false</initialOrientationAsReference>
+    </plugin>
+    <pose>0 0 0 0 0 0</pose>
+  </sensor>
 </gazebo>
 </robot>

Commit message: Added the camera sensor to the smile mobile robot simulation model.

File: smile_mobile_sim_ws/src/smile_mobile_description/urdf/smile.urdf.xacro (robot description, xacro)
@@ -152,12 +152,4 @@
     <dynamics damping="1.5"/>
   </joint>
-  <!--A small link to connect the IMU to the chassis-->
-  <link name="imu_link">
-  </link>
-  <joint name="chassis_to_imu_link" type="fixed">
-    <parent link="chassis"/>
-    <child link="imu_link"/>
-    <origin xyz="0.0 0.0 0.0"/>
-  </joint>
   <!-- Gazebo References for URDF model
   <gazebo reference="chassis">
@@ -234,4 +226,12 @@
   <mu2>0.5</mu2>
 </gazebo>
+<!--A small link to connect the IMU to the chassis-->
+<link name="imu_link">
+</link>
+<joint name="chassis_to_imu_link" type="fixed">
+  <parent link="chassis"/>
+  <child link="imu_link"/>
+  <origin xyz="0.0 0.0 0.0"/>
+</joint>
 <!--IMU Sensor Plugin-->
 <gazebo reference="imu_link">
@@ -255,3 +255,64 @@
   </sensor>
 </gazebo>
+<!--Camera sensor-->
+<link name="camera_link">
+  <collision>
+    <origin xyz="0 0 0" rpy="0 0 0"/>
+    <geometry>
+      <box size="0.05 0.02 0.02"/>
+    </geometry>
+  </collision>
+  <visual>
+    <origin xyz="0 0 0" rpy="0 0 0"/>
+    <geometry>
+      <box size="0.05 0.02 0.02"/>
+    </geometry>
+    <material name="black"/>
+  </visual>
+</link>
+<joint name="chassis_to_camera_link" type="fixed">
+  <axis xyz="0 0 0"/>
+  <origin xyz="0 ${chassis_length/2.0} ${chassis_height/2.0 + 0.01}" rpy="0 0 1.57"/>
+  <parent link="chassis"/>
+  <child link="camera_link"/>
+</joint>
+<gazebo reference="camera_link">
+   <sensor type="camera" name="camera1">
+     <update_rate>30.0</update_rate>
+     <camera name="head">
+       <horizontal_fov>1.3962634</horizontal_fov>
+       <image>
+         <width>800</width>
+         <height>800</height>
+         <format>R8G8B8</format>
+       </image>
+       <clip>
+         <near>0.02</near>
+         <far>300</far>
+       </clip>
+       <noise>
+         <type>gaussian</type>
+         <!-- Noise is sampled independently per pixel on each frame.
+              That pixel's noise value is added to each of its color
+              channels, which at that point lie in the range [0,1]. -->
+         <mean>0.0</mean>
+         <stddev>0.007</stddev>
+       </noise>
+     </camera>
+     <plugin name="camera_controller" filename="libgazebo_ros_camera.so">
+       <alwaysOn>true</alwaysOn>
+       <updateRate>0.0</updateRate>
+       <cameraName>smile/camera1</cameraName>
+       <imageTopicName>image_raw</imageTopicName>
+       <cameraInfoTopicName>camera_info</cameraInfoTopicName>
+       <frameName>camera_link</frameName>
+       <hackBaseline>0.07</hackBaseline>
+       <distortionK1>0.0</distortionK1>
+       <distortionK2>0.0</distortionK2>
+       <distortionK3>0.0</distortionK3>
+       <distortionT1>0.0</distortionT1>
+       <distortionT2>0.0</distortionT2>
+     </plugin>
+   </sensor>
+ </gazebo>
 </robot>

Commit message: Fixed the PID control and movement controller. PID's for simulation are tuned and work well! Also edited the Robot model so it faces the correct direction.

File: smile_mobile_sim_ws/src/smile_mobile_description/urdf/smile.urdf.xacro (robot description, xacro)
@@ -16,10 +16,10 @@
     <visual>
       <geometry>
-        <box size="${chassis_width} ${chassis_length} ${chassis_height}"/>
-      </geometry>
-    </visual>
-    <collision>
-      <geometry>
-        <box size="${chassis_width} ${chassis_length} ${chassis_height}"/>
+        <box size="${chassis_length} ${chassis_width} ${chassis_height}"/>
+      </geometry>
+    </visual>
+    <collision>
+      <geometry>
+        <box size="${chassis_length} ${chassis_width} ${chassis_height}"/>
       </geometry>
     </collision>
@@ -42,19 +42,19 @@
         <cylinder length="${wheel_width}" radius="${wheel_radius}"/>
       </geometry>
-      <origin rpy="0 ${pi_div_2} 0" xyz="${-1 * wheel_width / 2} 0 0"/>
-    </visual>
-    <collision>
-      <geometry>
-        <cylinder length="${wheel_width}" radius="${wheel_radius}"/>
-      </geometry>
-      <origin rpy="0 ${pi_div_2} 0" xyz="${-1 * wheel_width / 2} 0 0"/>
+      <origin rpy="0 ${pi_div_2} ${pi_div_2}" xyz="0 ${wheel_width / 2} 0"/>
+    </visual>
+    <collision>
+      <geometry>
+        <cylinder length="${wheel_width}" radius="${wheel_radius}"/>
+      </geometry>
+      <origin rpy="0 ${pi_div_2} ${pi_div_2}" xyz="0 ${wheel_width / 2} 0"/>
     </collision>
     <inertial>
       <mass value="${wheel_mass}"/>
       <inertia
-        ixx="${wheel_mass / 2.0 * wheel_radius * wheel_radius}" ixy="0.0" ixz="0.0"
-        iyy="0.01" iyz="0.0"
+        ixx="0.01" ixy="0.0" ixz="0.0"
+        iyy="${wheel_mass / 2.0 * wheel_radius * wheel_radius}" iyz="0.0"
         izz="0.01"/>
-      <origin rpy="0 ${pi_div_2} 0" xyz="${-1 * wheel_width / 2} 0 0"/>
+      <origin rpy="0 ${pi_div_2} ${pi_div_2}" xyz="0 ${wheel_width / 2} 0"/>
     </inertial>
   </link>
@@ -62,5 +62,6 @@
     <parent link="chassis"/>
     <child link="left_front_wheel"/>
-    <origin xyz="${-1 * chassis_width / 2} ${(chassis_length / 2) - wheel_pos_offset} 0 "/>
+    <origin xyz="${(chassis_length / 2) - wheel_pos_offset} ${chassis_width / 2} 0 "/>
+    <axis xyz="0 1 0"/>
     <dynamics damping="1.5"/>
   </joint>
@@ -71,19 +72,19 @@
         <cylinder length="${wheel_width}" radius="${wheel_radius}"/>
       </geometry>
-      <origin rpy="0 ${pi_div_2} 0" xyz="${wheel_width / 2} 0 0"/>
-    </visual>
-    <collision>
-      <geometry>
-        <cylinder length="${wheel_width}" radius="${wheel_radius}"/>
-      </geometry>
-      <origin rpy="0 ${pi_div_2} 0" xyz="${wheel_width / 2} 0 0"/>
+      <origin rpy="0 ${pi_div_2} ${pi_div_2}" xyz="0 ${-1*wheel_width / 2} 0"/>
+    </visual>
+    <collision>
+      <geometry>
+        <cylinder length="${wheel_width}" radius="${wheel_radius}"/>
+      </geometry>
+      <origin rpy="0 ${pi_div_2} ${pi_div_2}" xyz="0 ${-1*wheel_width / 2} 0"/>
     </collision>
     <inertial>
       <mass value="${wheel_mass}"/>
       <inertia
-        ixx="${wheel_mass / 2.0 * wheel_radius * wheel_radius}" ixy="0.0" ixz="0.0"
-        iyy="0.01" iyz="0.0"
+        ixx="0.01" ixy="0.0" ixz="0.0"
+        iyy="${wheel_mass / 2.0 * wheel_radius * wheel_radius}" iyz="0.0"
         izz="0.01"/>
-      <origin rpy="0 ${pi_div_2} 0" xyz="${wheel_width / 2} 0 0"/>
+      <origin rpy="0 ${pi_div_2} ${pi_div_2}" xyz="0 ${-1*wheel_width / 2} 0"/>
     </inertial>
   </link>
@@ -91,5 +92,6 @@
     <parent link="chassis"/>
     <child link="right_front_wheel"/>
-    <origin xyz="${chassis_width / 2} ${(chassis_length / 2) - wheel_pos_offset} 0 "/>
+    <origin xyz="${(chassis_length / 2) - wheel_pos_offset} ${-1 * chassis_width / 2} 0 "/>
+    <axis xyz="0 1 0"/>
     <dynamics damping="1.5"/>
   </joint>
@@ -100,19 +102,19 @@
         <cylinder length="${wheel_width}" radius="${wheel_radius}"/>
       </geometry>
-      <origin rpy="0 ${pi_div_2} 0" xyz="${-1 * wheel_width / 2} 0 0"/>
-    </visual>
-    <collision>
-      <geometry>
-        <cylinder length="${wheel_width}" radius="${wheel_radius}"/>
-      </geometry>
-      <origin rpy="0 ${pi_div_2} 0" xyz="${-1 * wheel_width / 2} 0 0"/>
+      <origin rpy="0 ${pi_div_2} ${pi_div_2}" xyz="0 ${wheel_width / 2} 0"/>
+    </visual>
+    <collision>
+      <geometry>
+        <cylinder length="${wheel_width}" radius="${wheel_radius}"/>
+      </geometry>
+      <origin rpy="0 ${pi_div_2} ${pi_div_2}" xyz="0 ${wheel_width / 2} 0"/>
     </collision>
     <inertial>
       <mass value="${wheel_mass}"/>
       <inertia
-        ixx="${wheel_mass / 2.0 * wheel_radius * wheel_radius}" ixy="0.0" ixz="0.0"
-        iyy="0.01" iyz="0.0"
+        ixx="0.01" ixy="0.0" ixz="0.0"
+        iyy="${wheel_mass / 2.0 * wheel_radius * wheel_radius}" iyz="0.0"
         izz="0.01"/>
-      <origin rpy="0 ${pi_div_2} 0" xyz="${-1 * wheel_width / 2} 0 0"/>
+      <origin rpy="0 ${pi_div_2} ${pi_div_2}" xyz="0 ${wheel_width / 2} 0"/>
     </inertial>
   </link>
@@ -120,5 +122,6 @@
     <parent link="chassis"/>
     <child link="left_back_wheel"/>
-    <origin xyz="${-1 * chassis_width / 2} ${-1 *(chassis_length / 2) + wheel_pos_offset} 0 "/>
+    <origin xyz="${(-1* chassis_length / 2) + wheel_pos_offset} ${chassis_width / 2} 0 "/>
+    <axis xyz="0 1 0"/>
     <dynamics damping="1.5"/>
   </joint>
@@ -129,19 +132,19 @@
         <cylinder length="${wheel_width}" radius="${wheel_radius}"/>
       </geometry>
-      <origin rpy="0 ${pi_div_2} 0" xyz="${wheel_width / 2} 0 0"/>
-    </visual>
-    <collision>
-      <geometry>
-        <cylinder length="${wheel_width}" radius="${wheel_radius}"/>
-      </geometry>
-      <origin rpy="0 ${pi_div_2} 0" xyz="${wheel_width / 2} 0 0"/>
+      <origin rpy="0 ${pi_div_2} ${pi_div_2}" xyz="0 ${-1*wheel_width / 2} 0"/>
+    </visual>
+    <collision>
+      <geometry>
+        <cylinder length="${wheel_width}" radius="${wheel_radius}"/>
+      </geometry>
+      <origin rpy="0 ${pi_div_2} ${pi_div_2}" xyz="0 ${-1*wheel_width / 2} 0"/>
     </collision>
     <inertial>
       <mass value="${wheel_mass}"/>
       <inertia
-        ixx="${wheel_mass / 2.0 * wheel_radius * wheel_radius}" ixy="0.0" ixz="0.0"
-        iyy="0.01" iyz="0.0"
+        ixx="0.01" ixy="0.0" ixz="0.0"
+        iyy="${wheel_mass / 2.0 * wheel_radius * wheel_radius}" iyz="0.0"
         izz="0.01"/>
-      <origin rpy="0 ${pi_div_2} 0" xyz="${wheel_width / 2} 0 0"/>
+      <origin rpy="0 ${pi_div_2} ${pi_div_2}" xyz="0 ${-1*wheel_width / 2} 0"/>
     </inertial>
   </link>
@@ -149,5 +152,6 @@
     <parent link="chassis"/>
     <child link="right_back_wheel"/>
-    <origin xyz="${chassis_width / 2} ${-1*(chassis_length / 2) + wheel_pos_offset} 0 "/>
+    <origin xyz="${(-1*chassis_length / 2) + wheel_pos_offset} ${-1 * chassis_width / 2} 0 "/>
+    <axis xyz="0 1 0"/>
     <dynamics damping="1.5"/>
   </joint>
@@ -273,5 +277,5 @@
 <joint name="chassis_to_camera_link" type="fixed">
   <axis xyz="0 0 0"/>
-  <origin xyz="0 ${chassis_length/2.0} ${chassis_height/2.0 + 0.01}" rpy="0 0 1.57"/>
+  <origin xyz="${chassis_length/2.0} 0 ${chassis_height/2.0 + 0.01}" rpy="0 0 0"/>
   <parent link="chassis"/>
   <child link="camera_link"/>

Commit message: Made a new sensor mount on the urdf simulation model of the robot to allow the camera to sit higher. Still need to test the lane detector.

File: smile_mobile_sim_ws/src/smile_mobile_description/urdf/smile.urdf.xacro (robot description, xacro)
@@ -10,4 +10,6 @@
   <xacro:property name="wheel_pos_offset" value=".0254"/>
   <xacro:property name="wheel_mass" value="0.5"/>
+  <xacro:property name="sensor_mount_width" value="0.15"/>
+  <xacro:property name="sensor_mount_height" value="0.2"/>
   <xacro:property name="pi_div_2" value="1.57075"/>
   <link name="base_link"/>
@@ -260,9 +262,9 @@
 </gazebo>
 <!--Camera sensor-->
-<link name="camera_link">
-  <collision>
+<link name="sensor_mount">
+   <collision>
     <origin xyz="0 0 0" rpy="0 0 0"/>
     <geometry>
-      <box size="0.05 0.02 0.02"/>
+        <box size="${sensor_mount_width} ${sensor_mount_width} ${sensor_mount_height}"/>
     </geometry>
   </collision>
@@ -270,12 +272,33 @@
     <origin xyz="0 0 0" rpy="0 0 0"/>
     <geometry>
-      <box size="0.05 0.02 0.02"/>
+      <box size="${sensor_mount_width} ${sensor_mount_width} ${sensor_mount_height}"/>
     </geometry>
     <material name="black"/>
   </visual>
 </link>
-<joint name="chassis_to_camera_link" type="fixed">
+<joint name="chassis_to_sensor_mount" type="fixed">
+    <axis xyz="0 0 0"/>
+    <origin xyz="0 0 ${(chassis_height / 2.0) + (sensor_mount_height/2.0)}" rpy="0 0 0"/>
+    <parent link="chassis"/>
+    <child link="sensor_mount"/>
+</joint>
+<xacro:property name="camera_dim" value="0.02"/>
+<link name="camera_link">
+  <collision>
+    <origin xyz="${camera_dim} 0 0" rpy="0 0 0"/>
+    <geometry>
+        <box size="${camera_dim} ${camera_dim} ${camera_dim}"/>
+    </geometry>
+  </collision>
+  <visual>
+    <origin xyz="${camera_dim} 0 0" rpy="0 0 0"/>
+    <geometry>
+       <box size="${camera_dim} ${camera_dim} ${camera_dim}"/>
+    </geometry>
+  </visual>
+</link>
+<joint name="sensor_mount_to_camera_link" type="fixed">
   <axis xyz="0 0 0"/>
-  <origin xyz="${chassis_length/2.0} 0 ${chassis_height/2.0 + 0.01}" rpy="0 0 0"/>
+  <origin xyz="${sensor_mount_width/2.0} 0 ${3.0*sensor_mount_height / 4.0}" rpy="0 0 0"/>
   <parent link="chassis"/>
   <child link="camera_link"/>
