Commit message: Added the scaling factor to the robot urdf. However, the robots PIDs will need to be retunned if the scale is changed.

File: smile_mobile_sim_ws/src/smile_mobile_description/urdf/smile.urdf.xacro (robot description, xacro)
@@ -1,15 +1,16 @@
 <?xml version="1.0"?>
 <robot name="smile" xmlns:xacro="http//www.ros.org/wiki/xacro">
-  <!--chassis Dimension [9" 10.5" 1.32"]-->
-  <xacro:property name="chassis_width" value="0.2286"/>
-  <xacro:property name="chassis_length" value="0.2667"/>
-  <xacro:property name="chassis_height" value="0.033528"/>
-  <xacro:property name="chassis_mass" value="1.0"/>
-  <xacro:property name="wheel_radius" value="0.06858"/>
-  <xacro:property name="wheel_width" value="0.0254"/>
-  <xacro:property name="wheel_pos_offset" value=".0254"/>
-  <xacro:property name="wheel_mass" value="0.5"/>
-  <xacro:property name="sensor_mount_width" value="0.15"/>
-  <xacro:property name="sensor_mount_height" value="0.2"/>
+   <xacro:property name="scale" value="3.0"/>
+   <!--chassis Dimension [9" 10.5" 1.32"]-->
+   <xacro:property name="chassis_width" value="${scale * 0.2286}"/>
+   <xacro:property name="chassis_length" value="${scale * 0.2667}"/>
+   <xacro:property name="chassis_height" value="${scale * 0.033528}"/>
+   <xacro:property name="chassis_mass" value="${scale * 1.0}"/>
+   <xacro:property name="wheel_radius" value="${scale * 0.06858}"/>
+   <xacro:property name="wheel_width" value="${scale * 0.0254}"/>
+   <xacro:property name="wheel_pos_offset" value="${scale * 0.0254}"/>
+   <xacro:property name="wheel_mass" value="${scale * 0.5}"/>
+   <xacro:property name="sensor_mount_width" value="${scale * 0.15}"/>
+   <xacro:property name="sensor_mount_height" value="${scale * 0.2}"/>
   <xacro:property name="pi_div_2" value="1.57075"/>
   <link name="base_link"/>

Commit message: Done with the whole flow

File: smile_mobile_sim_ws/src/smile_mobile_description/urdf/smile.urdf.xacro (robot description, xacro)
@@ -12,5 +12,5 @@
    <xacro:property name="wheel_mass" value="${scale * 0.5}"/>
    <xacro:property name="sensor_mount_width" value="${scale * 0.15}"/>
-   <xacro:property name="sensor_mount_height" value="${scale * 0.2}"/>
+   <xacro:property name="sensor_mount_height" value="${scale * 0.06}"/>
   <xacro:property name="pi_div_2" value="1.57075"/>
   <link name="base_link"/>
